Commit message: make odom - wheel tf happen : modify launch files

File: src/alfred_sim/description/gazebo_control.xacro (robot description, xacro)
@@ -1,29 +1,23 @@
 <?xml version="1.0"?>
 <robot xmlns:xacro="http://www.ros.org/wiki/xacro">
-    <gazebo>
-        <plugin name="gz::sim::systems::DiffDrive" filename="gz-sim-diff-drive-system">
-            <!-- Wheel Information -->
-            <left_joint>left_wheel_joint</left_joint>
-            <right_joint>right_wheel_joint</right_joint>
-            <wheel_separation>0.600</wheel_separation>
-            <wheel_radius>0.075</wheel_radius>
-            <!-- Limits -->
-            <!-- <max_wheel_torque>200</max_wheel_torque> -->
-            <max_linear_acceleration>0.33</max_linear_acceleration>
-            <!-- Input -->
-            <topic>cmd_vel</topic>
-            <!-- Output -->
-            <frame_id>odom</frame_id>
-            <child_frame_id>base_link</child_frame_id>
-            <odom_topic>odom</odom_topic>
-            <odom_publisher_frequency>30</odom_publisher_frequency>
-            <tf_topic>/tf</tf_topic>
-        </plugin>
-        <plugin filename="gz-sim-joint-state-publisher-system"
-            name="gz::sim::systems::JointStatePublisher">
-            <topic>joint_states</topic>
-            <joint_name>left_wheel_joint</joint_name>
-            <joint_name>right_wheel_joint</joint_name>
-        </plugin>
-    </gazebo>
+   <gazebo>
+      <plugin filename="gz-sim-diff-drive-system" name="gz::sim::systems::DiffDrive">
+         <right_joint>right_wheel_joint</right_joint>
+         <left_joint>left_wheel_joint</left_joint>
+         <wheel_separation>0.6</wheel_separation>
+         <wheel_radius>0.075</wheel_radius>
+         <max_linear_acceleration>0.33</max_linear_acceleration>
+         <topic>cmd_vel</topic>
+         <odom_topic>odom</odom_topic>
+         <frame_id>odom</frame_id>
+         <child_frame_id>base_link</child_frame_id>
+         <odom_publisher_frequency>100</odom_publisher_frequency>
+         <tf_topic>/tf</tf_topic>
+      </plugin>
+      <plugin filename="gz-sim-joint-state-publisher-system" name="gz::sim::systems::JointStatePublisher">
+         <topic>joint_states</topic>
+         <joint_name>right_wheel_joint</joint_name>
+         <joint_name>left_wheel_joint</joint_name>
+      </plugin>
+   </gazebo>
 </robot>

File: src/alfred_sim/description/robot_core.xacro (robot description, xacro)
@@ -6,12 +6,4 @@
     <xacro:include filename="material.xacro"/>
     <link name="base_link"></link>
-    <!-- BASE_FOOTPRINT LINK -->
-    <joint name="base_footprint_joint" type="fixed">
-        <parent link="base_link"/>
-        <child link="base_footprint"/>
-        <origin xyz="0 0 0" rpy="0 0 0"/>
-    </joint>
-    <link name="base_footprint">
-    </link>
     <!-- CHASSIS LINK -->
     <joint name="chassis_joint" type="fixed">
