Commit message: base_footprint link added for nav reference

File: src/alfred_sim/description/robot_core.xacro (robot description, xacro)
@@ -6,4 +6,11 @@
     <xacro:include filename="material.xacro"/>
     <link name="base_link"></link>
+    <link name="base_footprint"></link>
+    <!-- BASE_FOOTPRINT LINK -->
+    <joint name="base_footprint_joint" type="fixed">
+        <parent link="base_link"/>
+        <child link="base_footprint"/>
+        <origin xyz="0 0 0"/>
+    </joint>
     <!-- CHASSIS LINK -->
     <joint name="chassis_joint" type="fixed">
