Commit message: modify to fit/ tune parameters for the test body

File: src/alfred_sim/description/lidar.xacro (robot description, xacro)
@@ -5,5 +5,5 @@
      <parent link="chassis"/>
      <child link="laser_frame"/>
-     <origin xyz="0.420 0 0.200" rpy="0 0 0"/>
+     <origin xyz="0.520 0 0.280" rpy="0 0 0"/>
    </joint>
    <link name="laser_frame">

File: src/alfred_sim/description/properties.xacro (robot description, xacro)
@@ -2,18 +2,18 @@
 <robot xmlns:xacro="http://www.ros.org/wiki/xacro">
 <!-- contains all the properties of the bot, one stop shop to change all dimentions  -->
-    <xacro:property name="chassis_length" value="0.500"/>
+    <xacro:property name="chassis_length" value="0.560"/>
     <xacro:property name="chassis_width" value="0.600"/>
-    <xacro:property name="chassis_height" value="0.200"/>
+    <xacro:property name="chassis_height" value="0.260"/>
     <xacro:property name="chassis_mass" value="1.0"/>
-    <xacro:property name="wheel_radius" value="0.075"/>
+    <xacro:property name="wheel_radius" value="0.12"/>
     <xacro:property name="wheel_thickness" value="0.026"/>
     <xacro:property name="wheel_mass" value="0.05"/>
-    <xacro:property name="wheel_offset_x" value="0.250"/>
+    <xacro:property name="wheel_offset_x" value="0.170"/>
     <xacro:property name="wheel_offset_y" value="0.300"/>
     <xacro:property name="wheel_offset_z" value="0"/>
-    <xacro:property name="caster_wheel_radius" value="0.0375"/>
+    <xacro:property name="caster_wheel_radius" value="0.06"/>
     <xacro:property name="caster_wheel_mass" value="0.01"/>
-    <xacro:property name="caster_wheel_offset_x" value="0.200"/>
-    <xacro:property name="caster_wheel_offset_y" value="0.250"/>
-    <xacro:property name="caster_wheel_offset_z" value="0.037"/>
+    <xacro:property name="caster_wheel_offset_x" value="0.290"/>
+    <xacro:property name="caster_wheel_offset_y" value="0"/>
+    <xacro:property name="caster_wheel_offset_z" value="0.06"/>
 </robot>

File: src/alfred_sim/description/robot_core.xacro (robot description, xacro)
@@ -92,11 +92,11 @@
         <material>Gazebo/Blue</material>
     </gazebo>
-<!-- CASTER WHEEL LINK Front-Left-->
-    <joint name="caster_wheel_fl_joint" type="fixed">
+<!-- CASTER WHEEL -->
+    <joint name="caster_wheel_joint" type="fixed">
         <parent link="base_link"/>
-        <child link="caster_wheel_fl"/>
+        <child link="caster_wheel"/>
         <origin xyz="${caster_wheel_offset_x} ${caster_wheel_offset_y} -${caster_wheel_offset_z}"/>
     </joint>
-    <link name="caster_wheel_fl">
+    <link name="caster_wheel">
         <visual>
             <geometry>
@@ -114,89 +114,5 @@
         </xacro:inertial_sphere>
     </link>
-    <gazebo reference="caster_wheel_fl">
-        <material>Gazebo/White</material>
-        <!--the lesser the value the lesser the friction-->
-        <mu1 value="0.000000000000000001"/>
-        <mu2 value="0.000000000000000001"/>
-    </gazebo>
-<!-- CASTER WHEEL LINK Front-Right-->
-    <joint name="caster_wheel_fr_joint" type="fixed">
-        <parent link="base_link"/>
-        <child link="caster_wheel_fr"/>
-        <origin xyz="${caster_wheel_offset_x} -${caster_wheel_offset_y} -${caster_wheel_offset_z}"/>
-    </joint>
-    <link name="caster_wheel_fr">
-        <visual>
-            <geometry>
-                <sphere radius="${caster_wheel_radius}"/>
-            </geometry>
-            <material name="white"/>
-        </visual>
-        <collision>
-            <geometry>
-                <sphere radius="${caster_wheel_radius}"/>
-            </geometry>
-        </collision>
-        <xacro:inertial_sphere mass="${caster_wheel_mass}" radius="${caster_wheel_radius}">
-            <origin xyz="0 0 0" rpy="0 0 0"/>
-        </xacro:inertial_sphere>
-    </link>
-    <gazebo reference="caster_wheel_fr">
-        <material>Gazebo/White</material>
-        <!--the lesser the value the lesser the friction-->
-        <mu1 value="0.000000000000000001"/>
-        <mu2 value="0.000000000000000001"/>
-    </gazebo>
-<!-- CASTER WHEEL LINK Back-Left-->
-    <joint name="caster_wheel_bl_joint" type="fixed">
-        <parent link="base_link"/>
-        <child link="caster_wheel_bl"/>
-        <origin xyz="-${caster_wheel_offset_x} ${caster_wheel_offset_y} -${caster_wheel_offset_z}"/>
-    </joint>
-    <link name="caster_wheel_bl">
-        <visual>
-            <geometry>
-                <sphere radius="${caster_wheel_radius}"/>
-            </geometry>
-            <material name="white"/>
-        </visual>
-        <collision>
-            <geometry>
-                <sphere radius="${caster_wheel_radius}"/>
-            </geometry>
-        </collision>
-        <xacro:inertial_sphere mass="${caster_wheel_mass}" radius="${caster_wheel_radius}">
-            <origin xyz="0 0 0" rpy="0 0 0"/>
-        </xacro:inertial_sphere>
-    </link>
-    <gazebo reference="caster_wheel_bl">
-        <material>Gazebo/White</material>
-        <!--the lesser the value the lesser the friction-->
-        <mu1 value="0.000000000000000001"/>
-        <mu2 value="0.000000000000000001"/>
-    </gazebo>
-<!-- CASTER WHEEL LINK Back-Right-->
-    <joint name="caster_wheel_br_joint" type="fixed">
-        <parent link="base_link"/>
-        <child link="caster_wheel_br"/>
-        <origin xyz="-${caster_wheel_offset_x} -${caster_wheel_offset_y} -${caster_wheel_offset_z}"/>
-    </joint>
-    <link name="caster_wheel_br">
-        <visual>
-            <geometry>
-                <sphere radius="${caster_wheel_radius}"/>
-            </geometry>
-            <material name="white"/>
-        </visual>
-        <collision>
-            <geometry>
-                <sphere radius="${caster_wheel_radius}"/>
-            </geometry>
-        </collision>
-        <xacro:inertial_sphere mass="${caster_wheel_mass}" radius="${caster_wheel_radius}">
-            <origin xyz="0 0 0" rpy="0 0 0"/>
-        </xacro:inertial_sphere>
-    </link>
-    <gazebo reference="caster_wheel_br">
+    <gazebo reference="caster_wheel">
         <material>Gazebo/White</material>
         <!--the lesser the value the lesser the friction-->

Commit message: back to alfred dimentions

File: src/alfred_sim/description/lidar.xacro (robot description, xacro)
@@ -5,11 +5,11 @@
      <parent link="chassis"/>
      <child link="laser_frame"/>
-     <origin xyz="0.520 0 0.280" rpy="0 0 0"/>
+     <origin xyz="0.485 0 0.207" rpy="0 0 0"/>
    </joint>
    <link name="laser_frame">
       <visual>
-         <origin xyz="0 0 0.02"/>
+         <origin xyz="0 0 0"/>
          <geometry>
-            <cylinder length="0.04" radius="0.05"/>
+            <cylinder length="0.015" radius="0.026"/>
          </geometry>
          <material name="laser_material">
@@ -20,8 +20,8 @@
          <origin xyz="0 0 0"/>
          <geometry>
-            <cylinder length="0.04" radius="0.05"/>
+            <cylinder length="0.015" radius="0.026"/>
          </geometry>
       </collision>
-      <xacro:inertial_cylinder mass="0.1" length="0.04" radius="0.05">
+      <xacro:inertial_cylinder mass="0.1" length="0.015" radius="0.026">
          <origin xyz="0 0 0" rpy="0 0 0"/>
       </xacro:inertial_cylinder>

File: src/alfred_sim/description/properties.xacro (robot description, xacro)
@@ -2,18 +2,18 @@
 <robot xmlns:xacro="http://www.ros.org/wiki/xacro">
 <!-- contains all the properties of the bot, one stop shop to change all dimentions  -->
-    <xacro:property name="chassis_length" value="0.560"/>
+    <xacro:property name="chassis_length" value="0.520"/>
     <xacro:property name="chassis_width" value="0.600"/>
-    <xacro:property name="chassis_height" value="0.260"/>
+    <xacro:property name="chassis_height" value="0.200"/>
     <xacro:property name="chassis_mass" value="1.0"/>
-    <xacro:property name="wheel_radius" value="0.12"/>
-    <xacro:property name="wheel_thickness" value="0.026"/>
+    <xacro:property name="wheel_radius" value="0.075"/>
+    <xacro:property name="wheel_thickness" value="0.051"/>
     <xacro:property name="wheel_mass" value="0.05"/>
-    <xacro:property name="wheel_offset_x" value="0.170"/>
+    <xacro:property name="wheel_offset_x" value="0.26"/>
     <xacro:property name="wheel_offset_y" value="0.300"/>
     <xacro:property name="wheel_offset_z" value="0"/>
-    <xacro:property name="caster_wheel_radius" value="0.06"/>
+    <xacro:property name="caster_wheel_radius" value="0.0375"/>
     <xacro:property name="caster_wheel_mass" value="0.01"/>
-    <xacro:property name="caster_wheel_offset_x" value="0.290"/>
-    <xacro:property name="caster_wheel_offset_y" value="0"/>
-    <xacro:property name="caster_wheel_offset_z" value="0.06"/>
+    <xacro:property name="caster_wheel_offset_x" value="0.22"/>
+    <xacro:property name="caster_wheel_offset_y" value="0.26"/>
+    <xacro:property name="caster_wheel_offset_z" value="0.0375"/>
 </robot>

File: src/alfred_sim/description/robot_core.xacro (robot description, xacro)
@@ -1,122 +1,206 @@
 <?xml version="1.0"?>
 <robot xmlns:xacro="http://www.ros.org/wiki/xacro">
-<!-- This will contain the core structure defined.  -->
-    <xacro:include filename="inertial_macros.xacro"/>
-    <xacro:include filename="properties.xacro"/>
-    <xacro:include filename="material.xacro"/>
-    <link name="base_link"></link>
-    <link name="base_footprint"></link>
-    <!-- BASE_FOOTPRINT LINK -->
-    <joint name="base_footprint_joint" type="fixed">
-        <parent link="base_link"/>
-        <child link="base_footprint"/>
-        <origin xyz="0 0 0"/>
-    </joint>
-    <!-- CHASSIS LINK -->
-    <joint name="chassis_joint" type="fixed">
-        <parent link="base_link"/>
-        <child link="chassis"/>
-        <origin xyz="${-wheel_offset_x} 0 0"/>
-    </joint>
-    <link name="chassis">
-        <visual>
-            <origin xyz="${chassis_length/2} 0 ${chassis_height/2}"/>
-            <geometry>
-                <box size="${chassis_length} ${chassis_width} ${chassis_height}"/>
-            </geometry>
-            <material name="orange"/>
-        </visual>
-        <collision>
-            <origin xyz="${chassis_length/2} 0 ${chassis_height/2}"/>
-            <geometry>
-                <box size="${chassis_length} ${chassis_width} ${chassis_height}"/>
-            </geometry>
-        </collision>
-        <xacro:inertial_box mass="0.5" x="${chassis_length}" y="${chassis_width}" z="${chassis_height}">
-            <origin xyz="${chassis_length/2} 0 ${chassis_height/2}" rpy="0 0 0"/>
-        </xacro:inertial_box>
-    </link>
-    <gazebo reference="chassis">
-        <material>Gazebo/Orange</material>
-    </gazebo>
-    <!-- LEFT WHEEL LINK -->
-    <joint name="left_wheel_joint" type="continuous">
-        <parent link="base_link"/>
-        <child link="left_wheel"/>
-        <origin xyz="0 ${wheel_offset_y} 0" rpy="-${pi/2} 0 0" />
-        <axis xyz="0 0 1"/>
-    </joint>
-    <link name="left_wheel">
-        <visual>
-            <geometry>
-                <cylinder radius="${wheel_radius}" length="${wheel_thickness}"/>
-            </geometry>
-            <material name="blue"/>
-        </visual>
-        <collision>
-            <geometry>
-                <sphere radius="${wheel_radius}"/>
-            </geometry>
-        </collision>
-        <xacro:inertial_cylinder mass="${wheel_mass}" length="${wheel_thickness}" radius="${wheel_radius}">
-            <origin xyz="0 0 0" rpy="0 0 0"/>
-        </xacro:inertial_cylinder>
-    </link>
-    <gazebo reference="left_wheel">
-        <material>Gazebo/Blue</material>
-    </gazebo>
- <!-- RIGHT WHEEL LINK -->
-    <joint name="right_wheel_joint" type="continuous">
-        <parent link="base_link"/>
-        <child link="right_wheel"/>
-        <origin xyz="0 ${-wheel_offset_y} 0" rpy="${pi/2} 0 0" />
-        <axis xyz="0 0 -1"/>
-    </joint>
-    <link name="right_wheel">
-        <visual>
-            <geometry>
-                <cylinder radius="${wheel_radius}" length="${wheel_thickness}"/>
-            </geometry>
-            <material name="blue"/>
-        </visual>
-        <collision>
-            <geometry>
-                <sphere radius="${wheel_radius}"/>
-            </geometry>
-        </collision>
-        <xacro:inertial_cylinder mass="${wheel_mass}" length="${wheel_thickness}" radius="${wheel_radius}">
-            <origin xyz="0 0 0" rpy="0 0 0"/>
-        </xacro:inertial_cylinder>
-    </link>
-    <gazebo reference="right_wheel">
-        <material>Gazebo/Blue</material>
-    </gazebo>
-<!-- CASTER WHEEL -->
-    <joint name="caster_wheel_joint" type="fixed">
-        <parent link="base_link"/>
-        <child link="caster_wheel"/>
-        <origin xyz="${caster_wheel_offset_x} ${caster_wheel_offset_y} -${caster_wheel_offset_z}"/>
-    </joint>
-    <link name="caster_wheel">
-        <visual>
-            <geometry>
-                <sphere radius="${caster_wheel_radius}"/>
-            </geometry>
-            <material name="white"/>
-        </visual>
-        <collision>
-            <geometry>
-                <sphere radius="${caster_wheel_radius}"/>
-            </geometry>
-        </collision>
-        <xacro:inertial_sphere mass="${caster_wheel_mass}" radius="${caster_wheel_radius}">
-            <origin xyz="0 0 0" rpy="0 0 0"/>
-        </xacro:inertial_sphere>
-    </link>
-    <gazebo reference="caster_wheel">
-        <material>Gazebo/White</material>
-        <!--the lesser the value the lesser the friction-->
-        <mu1 value="0.000000000000000001"/>
-        <mu2 value="0.000000000000000001"/>
-    </gazebo>
-</robot>
+ <!-- This will contain the core structure defined.  -->
+     <xacro:include filename="inertial_macros.xacro"/>
+     <xacro:include filename="properties.xacro"/>
+     <xacro:include filename="material.xacro"/>
+     <link name="base_link"></link>
+     <link name="base_footprint"></link>
+     <!-- BASE_FOOTPRINT LINK -->
+     <joint name="base_footprint_joint" type="fixed">
+         <parent link="base_link"/>
+         <child link="base_footprint"/>
+         <origin xyz="0 0 0"/>
+     </joint>
+     <!-- CHASSIS LINK -->
+     <joint name="chassis_joint" type="fixed">
+         <parent link="base_link"/>
+         <child link="chassis"/>
+         <origin xyz="${-wheel_offset_x} 0 0"/>
+     </joint>
+     <link name="chassis">
+         <visual>
+             <origin xyz="${chassis_length/2} 0 ${chassis_height/2}"/>
+             <geometry>
+                 <box size="${chassis_length} ${chassis_width} ${chassis_height}"/>
+             </geometry>
+             <material name="orange"/>
+         </visual>
+         <collision>
+             <origin xyz="${chassis_length/2} 0 ${chassis_height/2}"/>
+             <geometry>
+                 <box size="${chassis_length} ${chassis_width} ${chassis_height}"/>
+             </geometry>
+         </collision>
+         <xacro:inertial_box mass="0.5" x="${chassis_length}" y="${chassis_width}" z="${chassis_height}">
+             <origin xyz="${chassis_length/2} 0 ${chassis_height/2}" rpy="0 0 0"/>
+         </xacro:inertial_box>
+     </link>
+     <gazebo reference="chassis">
+         <material>Gazebo/Orange</material>
+     </gazebo>
+     <!-- LEFT WHEEL LINK -->
+     <joint name="left_wheel_joint" type="continuous">
+         <parent link="base_link"/>
+         <child link="left_wheel"/>
+         <origin xyz="0 ${wheel_offset_y} 0" rpy="-${pi/2} 0 0" />
+         <axis xyz="0 0 1"/>
+     </joint>
+     <link name="left_wheel">
+         <visual>
+             <geometry>
+                 <cylinder radius="${wheel_radius}" length="${wheel_thickness}"/>
+             </geometry>
+             <material name="blue"/>
+         </visual>
+         <collision>
+             <geometry>
+                 <sphere radius="${wheel_radius}"/>
+             </geometry>
+         </collision>
+         <xacro:inertial_cylinder mass="${wheel_mass}" length="${wheel_thickness}" radius="${wheel_radius}">
+             <origin xyz="0 0 0" rpy="0 0 0"/>
+         </xacro:inertial_cylinder>
+     </link>
+     <gazebo reference="left_wheel">
+         <material>Gazebo/Blue</material>
+     </gazebo>
+  <!-- RIGHT WHEEL LINK -->
+     <joint name="right_wheel_joint" type="continuous">
+         <parent link="base_link"/>
+         <child link="right_wheel"/>
+         <origin xyz="0 ${-wheel_offset_y} 0" rpy="${pi/2} 0 0" />
+         <axis xyz="0 0 -1"/>
+     </joint>
+     <link name="right_wheel">
+         <visual>
+             <geometry>
+                 <cylinder radius="${wheel_radius}" length="${wheel_thickness}"/>
+             </geometry>
+             <material name="blue"/>
+         </visual>
+         <collision>
+             <geometry>
+                 <sphere radius="${wheel_radius}"/>
+             </geometry>
+         </collision>
+         <xacro:inertial_cylinder mass="${wheel_mass}" length="${wheel_thickness}" radius="${wheel_radius}">
+             <origin xyz="0 0 0" rpy="0 0 0"/>
+         </xacro:inertial_cylinder>
+     </link>
+     <gazebo reference="right_wheel">
+         <material>Gazebo/Blue</material>
+     </gazebo>
+ <!-- CASTER WHEEL LINK Front-Left-->
+     <joint name="caster_wheel_fl_joint" type="fixed">
+         <parent link="base_link"/>
+         <child link="caster_wheel_fl"/>
+         <origin xyz="${caster_wheel_offset_x} ${caster_wheel_offset_y} -${caster_wheel_offset_z}"/>
+     </joint>
+     <link name="caster_wheel_fl">
+         <visual>
+             <geometry>
+                 <sphere radius="${caster_wheel_radius}"/>
+             </geometry>
+             <material name="white"/>
+         </visual>
+         <collision>
+             <geometry>
+                 <sphere radius="${caster_wheel_radius}"/>
+             </geometry>
+         </collision>
+         <xacro:inertial_sphere mass="${caster_wheel_mass}" radius="${caster_wheel_radius}">
+             <origin xyz="0 0 0" rpy="0 0 0"/>
+         </xacro:inertial_sphere>
+     </link>
+     <gazebo reference="caster_wheel_fl">
+         <material>Gazebo/White</material>
+         <!--the lesser the value the lesser the friction-->
+         <mu1 value="0.000000000000000001"/>
+         <mu2 value="0.000000000000000001"/>
+     </gazebo>
+ <!-- CASTER WHEEL LINK Front-Right-->
+     <joint name="caster_wheel_fr_joint" type="fixed">
+         <parent link="base_link"/>
+         <child link="caster_wheel_fr"/>
+         <origin xyz="${caster_wheel_offset_x} -${caster_wheel_offset_y} -${caster_wheel_offset_z}"/>
+     </joint>
+     <link name="caster_wheel_fr">
+         <visual>
+             <geometry>
+                 <sphere radius="${caster_wheel_radius}"/>
+             </geometry>
+             <material name="white"/>
+         </visual>
+         <collision>
+             <geometry>
+                 <sphere radius="${caster_wheel_radius}"/>
+             </geometry>
+         </collision>
+         <xacro:inertial_sphere mass="${caster_wheel_mass}" radius="${caster_wheel_radius}">
+             <origin xyz="0 0 0" rpy="0 0 0"/>
+         </xacro:inertial_sphere>
+     </link>
+     <gazebo reference="caster_wheel_fr">
+         <material>Gazebo/White</material>
+         <!--the lesser the value the lesser the friction-->
+         <mu1 value="0.000000000000000001"/>
+         <mu2 value="0.000000000000000001"/>
+     </gazebo>
+ <!-- CASTER WHEEL LINK Back-Left-->
+     <joint name="caster_wheel_bl_joint" type="fixed">
+         <parent link="base_link"/>
+         <child link="caster_wheel_bl"/>
+         <origin xyz="-${caster_wheel_offset_x} ${caster_wheel_offset_y} -${caster_wheel_offset_z}"/>
+     </joint>
+     <link name="caster_wheel_bl">
+         <visual>
+             <geometry>
+                 <sphere radius="${caster_wheel_radius}"/>
+             </geometry>
+             <material name="white"/>
+         </visual>
+         <collision>
+             <geometry>
+                 <sphere radius="${caster_wheel_radius}"/>
+             </geometry>
+         </collision>
+         <xacro:inertial_sphere mass="${caster_wheel_mass}" radius="${caster_wheel_radius}">
+             <origin xyz="0 0 0" rpy="0 0 0"/>
+         </xacro:inertial_sphere>
+     </link>
+     <gazebo reference="caster_wheel_bl">
+         <material>Gazebo/White</material>
+         <!--the lesser the value the lesser the friction-->
+         <mu1 value="0.000000000000000001"/>
+         <mu2 value="0.000000000000000001"/>
+     </gazebo>
+ <!-- CASTER WHEEL LINK Back-Right-->
+     <joint name="caster_wheel_br_joint" type="fixed">
+         <parent link="base_link"/>
+         <child link="caster_wheel_br"/>
+         <origin xyz="-${caster_wheel_offset_x} -${caster_wheel_offset_y} -${caster_wheel_offset_z}"/>
+     </joint>
+     <link name="caster_wheel_br">
+         <visual>
+             <geometry>
+                 <sphere radius="${caster_wheel_radius}"/>
+             </geometry>
+             <material name="white"/>
+         </visual>
+         <collision>
+             <geometry>
+                 <sphere radius="${caster_wheel_radius}"/>
+             </geometry>
+         </collision>
+         <xacro:inertial_sphere mass="${caster_wheel_mass}" radius="${caster_wheel_radius}">
+             <origin xyz="0 0 0" rpy="0 0 0"/>
+         </xacro:inertial_sphere>
+     </link>
+     <gazebo reference="caster_wheel_br">
+         <material>Gazebo/White</material>
+         <!--the lesser the value the lesser the friction-->
+         <mu1 value="0.000000000000000001"/>
+         <mu2 value="0.000000000000000001"/>
+     </gazebo>
+ </robot>
