Commit message: test body params changed

File: src/alfred_robot/description/properties.xacro (robot description, xacro)
@@ -7,6 +7,6 @@
     <xacro:property name="chassis_mass" value="1.0"/>
     <xacro:property name="wheel_radius" value="0.12"/>
-    <xacro:property name="wheel_thickness" value="0.026"/>
-    <xacro:property name="wheel_mass" value="0.05"/>
+    <xacro:property name="wheel_thickness" value="0.08"/>
+    <xacro:property name="wheel_mass" value="2.0"/>
     <xacro:property name="wheel_offset_x" value="0.170"/>
     <xacro:property name="wheel_offset_y" value="0.300"/>

Commit message: make wheels come out of the bot, instead of half in half out

File: src/alfred_robot/description/properties.xacro (robot description, xacro)
@@ -10,5 +10,5 @@
     <xacro:property name="wheel_mass" value="2.0"/>
     <xacro:property name="wheel_offset_x" value="0.170"/>
-    <xacro:property name="wheel_offset_y" value="0.300"/>
+    <xacro:property name="wheel_offset_y" value="0.340"/>
     <xacro:property name="wheel_offset_z" value="0"/>
     <xacro:property name="caster_wheel_radius" value="0.06"/>
