Commit message: alfred sim works fine, add some tweaks to alfred robot package

File: src/alfred_robot/description/robot_core.xacro (robot description, xacro)
@@ -30,7 +30,4 @@
         </xacro:inertial_box>
     </link>
-    <gazebo reference="chassis">
-        <material>Gazebo/Orange</material>
-    </gazebo>
     <!-- LEFT WHEEL LINK -->
     <joint name="left_wheel_joint" type="continuous">
@@ -56,7 +53,4 @@
         </xacro:inertial_cylinder>
     </link>
-    <gazebo reference="left_wheel">
-        <material>Gazebo/Blue</material>
-    </gazebo>
  <!-- RIGHT WHEEL LINK -->
     <joint name="right_wheel_joint" type="continuous">
@@ -82,7 +76,4 @@
         </xacro:inertial_cylinder>
     </link>
-    <gazebo reference="right_wheel">
-        <material>Gazebo/Blue</material>
-    </gazebo>
 <!-- CASTER WHEEL LINK Front-Left-->
     <joint name="caster_wheel_fl_joint" type="fixed">
@@ -107,10 +98,4 @@
         </xacro:inertial_sphere>
     </link>
-    <gazebo reference="caster_wheel_fl">
-        <material>Gazebo/White</material>
-        <!--the lesser the value the lesser the friction-->
-        <mu1 value="0.000000000000000001"/>
-        <mu2 value="0.000000000000000001"/>
-    </gazebo>
 <!-- CASTER WHEEL LINK Front-Right-->
     <joint name="caster_wheel_fr_joint" type="fixed">
@@ -135,10 +120,4 @@
         </xacro:inertial_sphere>
     </link>
-    <gazebo reference="caster_wheel_fr">
-        <material>Gazebo/White</material>
-        <!--the lesser the value the lesser the friction-->
-        <mu1 value="0.000000000000000001"/>
-        <mu2 value="0.000000000000000001"/>
-    </gazebo>
 <!-- CASTER WHEEL LINK Back-Left-->
     <joint name="caster_wheel_bl_joint" type="fixed">
@@ -163,10 +142,4 @@
         </xacro:inertial_sphere>
     </link>
-    <gazebo reference="caster_wheel_bl">
-        <material>Gazebo/White</material>
-        <!--the lesser the value the lesser the friction-->
-        <mu1 value="0.000000000000000001"/>
-        <mu2 value="0.000000000000000001"/>
-    </gazebo>
 <!-- CASTER WHEEL LINK Back-Right-->
     <joint name="caster_wheel_br_joint" type="fixed">
@@ -191,9 +164,3 @@
         </xacro:inertial_sphere>
     </link>
-    <gazebo reference="caster_wheel_br">
-        <material>Gazebo/White</material>
-        <!--the lesser the value the lesser the friction-->
-        <mu1 value="0.000000000000000001"/>
-        <mu2 value="0.000000000000000001"/>
-    </gazebo>
 </robot>

File: src/alfred_robot/description/ros2_control.xacro (robot description, xacro)
@@ -2,7 +2,8 @@
 <robot xmlns:xacro="http://www.ros.org/wiki/xacro">
 <!-- ros 2 controller -->
-        <ros2_control name="GazeboSystem" type="system">
+        <ros2_control name="RealRobot" type="system">
             <hardware>
-                <plugin>gz_ros2_control/GazeboSimSystem</plugin>
+                <plugin>alfred_firmware/AlfredInterface</plugin>
+                <param name="port">/dev/ttyACM0</param>
             </hardware>
             <joint name="left_wheel_joint">
@@ -23,10 +24,4 @@
             </joint>
         </ros2_control>
-    <hardware>
-    <!-- Change the hardware plugin to be changed !!!!!!!!!!!!!!!!!!!!!!!!! -->
-        <plugin filename="gz_ros2_control-system" name="gz_ros2_control::GazeboSimROS2ControlPlugin">
-            <parameters>$(find alfred_sim)/config/my_controllers.yaml</parameters>
-        </plugin>
-    </hardware>
 </robot>
 <!-- to move the robot using twist keyboard, before connecting nav :  -->

Commit message: working commit

File: src/alfred_robot/description/robot_core.xacro (robot description, xacro)
@@ -37,12 +37,12 @@
         </xacro:inertial_box>
     </link>
-    <!-- LEFT WHEEL LINK -->
-    <joint name="left_wheel_joint" type="continuous">
+ <!-- RIGHT WHEEL LINK -->
+    <joint name="right_wheel_joint" type="continuous">
         <parent link="base_link"/>
-        <child link="left_wheel"/>
-        <origin xyz="0 ${wheel_offset_y} 0" rpy="-${pi/2} 0 0" />
-        <axis xyz="0 0 1"/>
+        <child link="right_wheel"/>
+        <origin xyz="0 ${-wheel_offset_y} 0" rpy="${pi/2} 0 0" />
+        <axis xyz="0 0 -1"/>
     </joint>
-    <link name="left_wheel">
+    <link name="right_wheel">
         <visual>
             <geometry>
@@ -60,12 +60,12 @@
         </xacro:inertial_cylinder>
     </link>
- <!-- RIGHT WHEEL LINK -->
-    <joint name="right_wheel_joint" type="continuous">
+    <!-- LEFT WHEEL LINK -->
+    <joint name="left_wheel_joint" type="continuous">
         <parent link="base_link"/>
-        <child link="right_wheel"/>
-        <origin xyz="0 ${-wheel_offset_y} 0" rpy="${pi/2} 0 0" />
-        <axis xyz="0 0 -1"/>
+        <child link="left_wheel"/>
+        <origin xyz="0 ${wheel_offset_y} 0" rpy="-${pi/2} 0 0" />
+        <axis xyz="0 0 1"/>
     </joint>
-    <link name="right_wheel">
+    <link name="left_wheel">
         <visual>
             <geometry>
